Commit message: modifications for urdfyangextension done

File: robot_specific_config/abb_irb1200_support/urdf/irb1200_5_90_macro.xacro (robot description, xacro)
@@ -2,7 +2,12 @@
 <robot xmlns:xacro="http://ros.org/wiki/xacro">
   <xacro:include filename="$(find abb_resources)/urdf/common_materials.xacro"/>
-  <xacro:macro name="abb_irb1200_5_90" params="prefix">
+  <xacro:macro name="abb_irb1200_5_90" params="parent id xyz:= '-1 1.2 2'">
     <!-- link list -->
-    <link name="${prefix}base_link">
+    <joint name="irb1200590_${id}_joint" type="fixed">
+      <parent link="${parent}" />
+      <origin xyz="${xyz}"/>
+      <child link="${id}base_link" />
+    </joint>
+    <link name="${id}base_link">
       <!-- See note 1 in package.xml about the inertial and mass values -->
       <inertial>
@@ -23,5 +28,5 @@
       </visual>
     </link>
-    <link name="${prefix}link_1">
+    <link name="${id}link_1">
       <!-- See note 1 in package.xml about the inertial and mass values -->
       <inertial>
@@ -42,5 +47,5 @@
       </visual>
     </link>
-    <link name="${prefix}link_2">
+    <link name="${id}link_2">
       <!-- See note 1 in package.xml about the inertial and mass values -->
       <inertial>
@@ -61,5 +66,5 @@
       </visual>
     </link>
-    <link name="${prefix}link_3">
+    <link name="${id}link_3">
       <!-- See note 1 in package.xml about the inertial and mass values -->
       <inertial>
@@ -80,5 +85,5 @@
       </visual>
     </link>
-    <link name="${prefix}link_4">
+    <link name="${id}link_4">
       <!-- See note 1 in package.xml about the inertial and mass values -->
       <inertial>
@@ -99,5 +104,5 @@
       </visual>
     </link>
-    <link name="${prefix}link_5">
+    <link name="${id}link_5">
       <!-- See note 1 in package.xml about the inertial and mass values -->
       <inertial>
@@ -118,5 +123,5 @@
       </visual>
     </link>
-    <link name="${prefix}link_6">
+    <link name="${id}link_6">
       <!-- See note 1 in package.xml about the inertial and mass values -->
       <inertial>
@@ -145,54 +150,54 @@
     <!-- end of link list -->
     <!-- joint list -->
-    <joint type="revolute" name="${prefix}joint_1">
+    <joint type="revolute" name="${id}joint_1">
       <origin xyz="0 0 0.3991" rpy="0 0 0"/>
       <axis xyz="0 0 1"/>
-      <parent link="${prefix}base_link"/>
-      <child link="${prefix}link_1"/>
+      <parent link="${id}base_link"/>
+      <child link="${id}link_1"/>
       <!-- See note 2 in package.xml about effort limits and dynamics values -->
       <limit effort="1000" lower="-2.967" upper="2.967" velocity="5.027"/>
       <dynamics damping="50.0" friction="1.0"/>
     </joint>
-    <joint type="revolute" name="${prefix}joint_2">
+    <joint type="revolute" name="${id}joint_2">
       <origin xyz="0 0 0" rpy="0 0 0"/>
       <axis xyz="0 1 0"/>
-      <parent link="${prefix}link_1"/>
-      <child link="${prefix}link_2"/>
+      <parent link="${id}link_1"/>
+      <child link="${id}link_2"/>
       <!-- See note 2 in package.xml about effort limits and dynamics values -->
       <limit effort="1000" lower="-1.745" upper="2.269" velocity="4.189"/>
       <dynamics damping="50.0" friction="1.0"/>
     </joint>
-    <joint type="revolute" name="${prefix}joint_3">
+    <joint type="revolute" name="${id}joint_3">
       <origin xyz="0 0 0.448" rpy="0 0 0"/>
       <axis xyz="0 1 0"/>
-      <parent link="${prefix}link_2"/>
-      <child link="${prefix}link_3"/>
+      <parent link="${id}link_2"/>
+      <child link="${id}link_3"/>
       <!-- See note 2 in package.xml about effort limits and dynamics values -->
       <limit effort="1000" lower="-3.491" upper="1.222" velocity="5.236"/>
       <dynamics damping="10.0" friction="1.0"/>
     </joint>
-    <joint type="revolute" name="${prefix}joint_4">
+    <joint type="revolute" name="${id}joint_4">
       <origin xyz="0 0 0.042" rpy="0 0 0"/>
       <axis xyz="1 0 0"/>
-      <parent link="${prefix}link_3"/>
-      <child link="${prefix}link_4"/>
+      <parent link="${id}link_3"/>
+      <child link="${id}link_4"/>
       <!-- See note 2 in package.xml about effort limits and dynamics values -->
       <limit effort="1000" lower="-4.712" upper="4.712" velocity="6.981"/>
       <dynamics damping="5.0" friction="1.0"/>
     </joint>
-    <joint type="revolute" name="${prefix}joint_5">
+    <joint type="revolute" name="${id}joint_5">
       <origin xyz="0.451 0 0" rpy="0 0 0"/>
       <axis xyz="0 1 0"/>
-      <parent link="${prefix}link_4"/>
-      <child link="${prefix}link_5"/>
+      <parent link="${id}link_4"/>
+      <child link="${id}link_5"/>
       <!-- See note 2 in package.xml about effort limits and dynamics values -->
       <limit effort="1000" lower="-2.269" upper="2.269" velocity="7.069"/>
       <dynamics damping="2.0" friction="1.0"/>
     </joint>
-    <joint type="revolute" name="${prefix}joint_6">
+    <joint type="revolute" name="${id}joint_6">
       <origin xyz="0.082 0 0" rpy="0 0 0"/>
       <axis xyz="1 0 0"/>
-      <parent link="${prefix}link_5"/>
-      <child link="${prefix}link_6"/>
+      <parent link="${id}link_5"/>
+      <child link="${id}link_6"/>
       <!-- See note 2 in package.xml about effort limits and dynamics values -->
       <limit effort="1000" lower="-6.283" upper="6.283" velocity="10.472"/>
@@ -201,24 +206,100 @@
     <!-- end of joint list -->
     <!-- ROS-Industrial 'base' frame- base_link to ABB World Coordinates transform -->
-    <link name="${prefix}base" />
-    <joint name="${prefix}base_link-base" type="fixed">
+    <link name="${id}base" />
+    <joint name="${id}base_link-base" type="fixed">
       <origin xyz="0 0 0" rpy="0 0 0"/>
-      <parent link="${prefix}base_link"/>
-      <child link="${prefix}base"/>
+      <parent link="${id}base_link"/>
+      <child link="${id}base"/>
     </joint>
     <!-- ROS-Industrial 'flange' frame- attachment point for EEF models -->
-    <link name="${prefix}flange"/>
-    <joint type="fixed" name="${prefix}joint_6-flange">
+    <link name="${id}flange"/>
+    <joint type="fixed" name="${id}joint_6-flange">
       <origin xyz="0 0 0" rpy="0 0 0"/>
-      <parent link="${prefix}link_6"/>
-      <child link="${prefix}flange"/>
+      <parent link="${id}link_6"/>
+      <child link="${id}flange"/>
     </joint>
     <!-- ROS-Industrial 'tool0' frame- all-zeros tool frame -->
-    <link name="${prefix}tool0" />
-    <joint name="${prefix}link_6-tool0" type="fixed">
+    <link name="${id}tool0" />
+    <joint name="${id}link_6-tool0" type="fixed">
       <origin xyz="0 0 0" rpy="0 ${radians(90)} 0" />
-      <parent link="${prefix}flange" />
-      <child link="${prefix}tool0" />
-    </joint>
+      <parent link="${id}flange" />
+      <child link="${id}tool0" />
+    </joint>
+       <yang>
+            <!-- Raspberry pi 4B network topology -->
+            <network>
+                <network-id>${L2_network_id}</network-id>
+                <supporting-network>
+                    <network-ref>${L1_network_id}</network-ref>
+                </supporting-network>
+                <node>
+                <node-id>${L2_id}</node-id>
+                <supporting-node>
+                    <network-ref>${L1_network_id}</network-ref>
+                    <node-ref>${L1_id}</node-ref>
+                </supporting-node>
+                <dl:device-layer-node-attributes xmlns:dl="urn:ietf:params:xml:ns:yang:device-layer">
+                    <dl:device-name>irb1200590</dl:device-name>
+                    <dl:device-type>robot-arm</dl:device-type>
+                </dl:device-layer-node-attributes>
+                <nt:termination-point xmlns:nt="urn:ietf:params:xml:ns:yang:ietf-network-topology">
+                    <nt:tp-id>_0</nt:tp-id>
+                    <nt:supporting-termination-point>
+                        <nt:network-ref>${L2_id}</nt:network-ref>
+                        <nt:node-ref>${L1_id}</nt:node-ref>
+                        <nt:tp-ref>eth_0</nt:tp-ref>
+                    </nt:supporting-termination-point>
+                    <dl:device-layer-termination-point-attributes xmlns:dl="urn:ietf:params:xml:ns:yang:device-layer">
+                        <dl:port-name>port1</dl:port-name>
+                        <dl:port-type>rj45</dl:port-type>
+                    </dl:device-layer-termination-point-attributes>
+                    <nl:network-layer-termination-point-attributes xmlns:nl="urn:ietf:params:xml:ns:yang:network-layer">
+                        <nl:interface-name>intf1</nl:interface-name>
+                        <nl:interface-type>ethernet</nl:interface-type>
+                        <nl:interface-status>up</nl:interface-status>
+                        <nl:mac-address>00:1A:2B:3C:4D:5E</nl:mac-address>
+                    </nl:network-layer-termination-point-attributes>
+                </nt:termination-point>
+                <nl:network-layer-node-attributes xmlns:nl="urn:ietf:params:xml:ns:yang:network-layer">
+                    <nl:node-name>netNode1</nl:node-name>
+                    <nl:node-type>generic</nl:node-type>
+                </nl:network-layer-node-attributes>
+                </node>
+                <dl:device-layer-topology xmlns:dl="urn:ietf:params:xml:ns:yang:device-layer">
+                    <dl:element>element2</dl:element>
+                </dl:device-layer-topology>
+                <nt:link xmlns:nt="urn:ietf:params:xml:ns:yang:ietf-network-topology">
+                    <nt:link-id>link1</nt:link-id>
+                    <nt:source>
+                        <nt:source-node>node1</nt:source-node>
+                        <nt:source-tp>tp1</nt:source-tp>
+                    </nt:source>
+                    <nt:destination>
+                        <nt:dest-node>node2</nt:dest-node>
+                        <nt:dest-tp>tp2</nt:dest-tp>
+                    </nt:destination>
+                    <nt:supporting-link>
+                        <nt:network-ref>network2</nt:network-ref>
+                        <nt:link-ref>link2</nt:link-ref>
+                    </nt:supporting-link>
+                    <dl:device-layer-link-attributes xmlns:dl="urn:ietf:params:xml:ns:yang:device-layer">
+                        <dl:physical-link-name>physLink1</dl:physical-link-name>
+                        <dl:physical-link-type>cat5e</dl:physical-link-type>
+                    </dl:device-layer-link-attributes>
+                    <nl:network-layer-link-attributes xmlns:nl="urn:ietf:params:xml:ns:yang:network-layer">
+                        <nl:link-name>netLink1</nl:link-name>
+                        <nl:link-type>3gpp-5g-qos-flow</nl:link-type>
+                        <nl:_5qi>1</nl:_5qi>
+                        <nl:gfbr>50</nl:gfbr>
+                        <nl:mfbr>100</nl:mfbr>
+                        <nl:pdb>20</nl:pdb>
+                        <nl:per>0</nl:per>
+                    </nl:network-layer-link-attributes>
+                </nt:link>
+                <nl:network-layer-topology xmlns:nl="urn:ietf:params:xml:ns:yang:network-layer">
+                    <nl:element>element3</nl:element>
+                </nl:network-layer-topology>
+            </network>
+        </yang>
   </xacro:macro>
 </robot>

File: robot_specific_config/abb_irb4600_support/urdf/irb4600_20_250_macro.xacro (robot description, xacro)
@@ -1,8 +1,13 @@
 <?xml version="1.0"?>
 <robot xmlns:xacro="http://ros.org/wiki/xacro">
-  <xacro:macro name="abb_irb4600_20_250" params="prefix">
+  <xacro:macro name="abb_irb4600_20_250" params="parent id xyz:= '6 6 6'">
     <xacro:include filename="$(find abb_resources)/urdf/common_materials.xacro"/>
+    <joint name="irb460020250_${id}_joint" type="fixed">
+      <parent link="${parent}" />
+      <origin xyz="${xyz}"/>
+      <child link="${id}base_link" />
+    </joint>
     <!-- link list -->
-    <link name="${prefix}base_link">
+    <link name="${id}base_link">
       <collision name="collision">
         <geometry>
@@ -18,5 +23,5 @@
       </visual>
     </link>
-    <link name="${prefix}link_1">
+    <link name="${id}link_1">
       <collision name="collision">
         <geometry>
@@ -32,5 +37,5 @@
       </visual>
     </link>
-    <link name="${prefix}link_2">
+    <link name="${id}link_2">
       <collision name="collision">
         <geometry>
@@ -46,5 +51,5 @@
       </visual>
     </link>
-    <link name="${prefix}link_3">
+    <link name="${id}link_3">
       <collision name="collision">
         <geometry>
@@ -60,5 +65,5 @@
       </visual>
     </link>
-    <link name="${prefix}link_4">
+    <link name="${id}link_4">
       <collision name="collision">
         <geometry>
@@ -74,5 +79,5 @@
       </visual>
     </link>
-    <link name="${prefix}link_5">
+    <link name="${id}link_5">
       <collision name="collision">
         <geometry>
@@ -88,5 +93,5 @@
       </visual>
     </link>
-    <link name="${prefix}link_6">
+    <link name="${id}link_6">
       <collision name="collision">
         <geometry>
@@ -104,68 +109,144 @@
     <!-- end of link list -->
     <!-- joint list -->
-    <joint type="revolute" name="${prefix}joint_1">
+    <joint type="revolute" name="${id}joint_1">
       <origin xyz="0 0 0.495" rpy="0 0 0"/>
       <axis xyz="0 0 1"/>
-      <parent link="${prefix}base_link"/>
-      <child link="${prefix}link_1"/>
+      <parent link="${id}base_link"/>
+      <child link="${id}link_1"/>
       <limit effort="0" lower="${radians(-180)}" upper="${radians(180)}" velocity="${radians(175)}"/>
     </joint>
-    <joint type="revolute" name="${prefix}joint_2">
+    <joint type="revolute" name="${id}joint_2">
       <origin xyz="0.175 0 0" rpy="0 0 0"/>
       <axis xyz="0 1 0"/>
-      <parent link="${prefix}link_1"/>
-      <child link="${prefix}link_2"/>
+      <parent link="${id}link_1"/>
+      <child link="${id}link_2"/>
       <limit effort="0" lower="${radians(-90)}" upper="${radians(150)}" velocity="${radians(175)}"/>
     </joint>
-    <joint type="revolute" name="${prefix}joint_3">
+    <joint type="revolute" name="${id}joint_3">
       <origin xyz="0 0 1.095" rpy="0 0 0"/>
       <axis xyz="0 1 0"/>
-      <parent link="${prefix}link_2"/>
-      <child link="${prefix}link_3"/>
+      <parent link="${id}link_2"/>
+      <child link="${id}link_3"/>
       <limit effort="0" lower="${radians(-180)}" upper="${radians(75)}" velocity="${radians(175)}"/>
     </joint>
-    <joint type="revolute" name="${prefix}joint_4">
+    <joint type="revolute" name="${id}joint_4">
       <origin xyz="0 0 0.175" rpy="0 0 0"/>
       <axis xyz="1 0 0"/>
-      <parent link="${prefix}link_3"/>
-      <child link="${prefix}link_4"/>
+      <parent link="${id}link_3"/>
+      <child link="${id}link_4"/>
       <limit effort="0" lower="${radians(-400)}" upper="${radians(400)}" velocity="${radians(360)}"/>
     </joint>
-    <joint type="revolute" name="${prefix}joint_5">
+    <joint type="revolute" name="${id}joint_5">
       <origin xyz="1.2305 0 0" rpy="0 0 0"/>
       <axis xyz="0 1 0"/>
-      <parent link="${prefix}link_4"/>
-      <child link="${prefix}link_5"/>
+      <parent link="${id}link_4"/>
+      <child link="${id}link_5"/>
       <limit effort="0" lower="${radians(-125)}" upper="${radians(120)}" velocity="${radians(360)}"/>
     </joint>
-    <joint type="revolute" name="${prefix}joint_6">
+    <joint type="revolute" name="${id}joint_6">
       <origin xyz="0.085 0 0" rpy="0 0 0"/>
       <axis xyz="1 0 0"/>
-      <parent link="${prefix}link_5"/>
-      <child link="${prefix}link_6"/>
+      <parent link="${id}link_5"/>
+      <child link="${id}link_6"/>
       <limit effort="0" lower="${radians(-400)}" upper="${radians(400)}" velocity="${radians(500)}"/>
     </joint>
     <!-- end of joint list -->
     <!-- ROS-Industrial 'base' frame- base_link to ABB World Coordinates transform -->
-    <link name="${prefix}base" />
-    <joint name="${prefix}base_link-base" type="fixed">
+    <link name="${id}base" />
+    <joint name="${id}base_link-base" type="fixed">
       <origin xyz="0 0 0" rpy="0 0 0"/>
-      <parent link="${prefix}base_link"/>
-      <child link="${prefix}base"/>
+      <parent link="${id}base_link"/>
+      <child link="${id}base"/>
     </joint>
     <!-- ROS-Industrial 'flange' frame- attachment point for EEF models -->
-    <link name="${prefix}flange"/>
-    <joint type="fixed" name="${prefix}joint_6-flange">
+    <link name="${id}flange"/>
+    <joint type="fixed" name="${id}joint_6-flange">
       <origin xyz="0 0 0" rpy="0 0 0"/>
-      <parent link="${prefix}link_6"/>
-      <child link="${prefix}flange"/>
+      <parent link="${id}link_6"/>
+      <child link="${id}flange"/>
     </joint>
     <!-- ROS-Industrial 'tool0' frame- all-zeros tool frame -->
-    <link name="${prefix}tool0" />
-    <joint name="${prefix}link_6-tool0" type="fixed">
+    <link name="${id}tool0" />
+    <joint name="${id}link_6-tool0" type="fixed">
       <origin xyz="0 0 0" rpy="0 ${radians(90)} 0" />
-      <parent link="${prefix}flange" />
-      <child link="${prefix}tool0" />
-    </joint>
+      <parent link="${id}flange" />
+      <child link="${id}tool0" />
+    </joint>
+       <yang>
+            <!-- Raspberry pi 4B network topology -->
+            <network>
+                <network-id>${L2_network_id}</network-id>
+                <supporting-network>
+                    <network-ref>${L1_network_id}</network-ref>
+                </supporting-network>
+                <node>
+                <node-id>${L2_id}</node-id>
+                <supporting-node>
+                    <network-ref>${L1_network_id}</network-ref>
+                    <node-ref>${L1_id}</node-ref>
+                </supporting-node>
+                <dl:device-layer-node-attributes xmlns:dl="urn:ietf:params:xml:ns:yang:device-layer">
+                    <dl:device-name>irb460020250</dl:device-name>
+                    <dl:device-type>robot-arm</dl:device-type>
+                </dl:device-layer-node-attributes>
+                <nt:termination-point xmlns:nt="urn:ietf:params:xml:ns:yang:ietf-network-topology">
+                    <nt:tp-id>_0</nt:tp-id>
+                    <nt:supporting-termination-point>
+                        <nt:network-ref>${L2_id}</nt:network-ref>
+                        <nt:node-ref>${L1_id}</nt:node-ref>
+                        <nt:tp-ref>eth_0</nt:tp-ref>
+                    </nt:supporting-termination-point>
+                    <dl:device-layer-termination-point-attributes xmlns:dl="urn:ietf:params:xml:ns:yang:device-layer">
+                        <dl:port-name>port1</dl:port-name>
+                        <dl:port-type>rj45</dl:port-type>
+                    </dl:device-layer-termination-point-attributes>
+                    <nl:network-layer-termination-point-attributes xmlns:nl="urn:ietf:params:xml:ns:yang:network-layer">
+                        <nl:interface-name>intf1</nl:interface-name>
+                        <nl:interface-type>ethernet</nl:interface-type>
+                        <nl:interface-status>up</nl:interface-status>
+                        <nl:mac-address>00:1A:2B:3C:4D:5E</nl:mac-address>
+                    </nl:network-layer-termination-point-attributes>
+                </nt:termination-point>
+                <nl:network-layer-node-attributes xmlns:nl="urn:ietf:params:xml:ns:yang:network-layer">
+                    <nl:node-name>netNode1</nl:node-name>
+                    <nl:node-type>generic</nl:node-type>
+                </nl:network-layer-node-attributes>
+                </node>
+                <dl:device-layer-topology xmlns:dl="urn:ietf:params:xml:ns:yang:device-layer">
+                    <dl:element>element2</dl:element>
+                </dl:device-layer-topology>
+                <nt:link xmlns:nt="urn:ietf:params:xml:ns:yang:ietf-network-topology">
+                    <nt:link-id>link1</nt:link-id>
+                    <nt:source>
+                        <nt:source-node>node1</nt:source-node>
+                        <nt:source-tp>tp1</nt:source-tp>
+                    </nt:source>
+                    <nt:destination>
+                        <nt:dest-node>node2</nt:dest-node>
+                        <nt:dest-tp>tp2</nt:dest-tp>
+                    </nt:destination>
+                    <nt:supporting-link>
+                        <nt:network-ref>network2</nt:network-ref>
+                        <nt:link-ref>link2</nt:link-ref>
+                    </nt:supporting-link>
+                    <dl:device-layer-link-attributes xmlns:dl="urn:ietf:params:xml:ns:yang:device-layer">
+                        <dl:physical-link-name>physLink1</dl:physical-link-name>
+                        <dl:physical-link-type>cat5e</dl:physical-link-type>
+                    </dl:device-layer-link-attributes>
+                    <nl:network-layer-link-attributes xmlns:nl="urn:ietf:params:xml:ns:yang:network-layer">
+                        <nl:link-name>netLink1</nl:link-name>
+                        <nl:link-type>3gpp-5g-qos-flow</nl:link-type>
+                        <nl:_5qi>1</nl:_5qi>
+                        <nl:gfbr>50</nl:gfbr>
+                        <nl:mfbr>100</nl:mfbr>
+                        <nl:pdb>20</nl:pdb>
+                        <nl:per>0</nl:per>
+                    </nl:network-layer-link-attributes>
+                </nt:link>
+                <nl:network-layer-topology xmlns:nl="urn:ietf:params:xml:ns:yang:network-layer">
+                    <nl:element>element3</nl:element>
+                </nl:network-layer-topology>
+            </network>
+        </yang>
   </xacro:macro>
 </robot>
